File: _saved_exercicio2.sch (KiCad schematic (older format))
At the start: 18 parts

Commit message: da ufal
Parts:
- added C? (x2): CP1, symbol CP1
- added C? (x2): C, symbol C
- added D?: LED, symbol LED
- added D?: D, symbol D
- added F?: Polyfuse, symbol Polyfuse
- added R?: R, symbol R
Connections:
- net GND: now also U?.2 (GND), C?.2, C?.2, C?.2, C?.2, D?.1 (K)
- net UVCC: now also F?.2
- net VCC: now also U?.5 (OUT), C?.1, C?.1, C?.1, R?.1
- net RAW: now reaches P?.1 (P1)
- net RAW: now also U?.1 (VIN), U?.3 (Enable), C?.1, D?.1 (K)
- new net: D?.2 (A), R?.2
- new net: D?.2 (A), F?.1
Other:
- moved on the sheet: U?
Changed lines of the file:
@@
 	2900 3850 3000 3850
 Wire Wire Line
-	4350 3500 4600 3500
-Wire Wire Line
-	4600 3500 5050 3500
+	4350 3500 5050 3500
 Wire Wire Line
 	5050 3500 5050 3650
 Wire Wire Line
-	4350 3800 4600 3800
-Wire Wire Line
-	4600 3800 5050 3800
+	4350 3800 5050 3800
 Wire Wire Line
 	5050 3800 5050 3750
@@
 Connection ~ 4600 3800
 Wire Wire Line
-	4050 3500 4050 3650
-Wire Wire Line
-	4050 3650 4050 3800
+	4050 3500 4050 3800
 Wire Wire Line
 	4000 3650 4050 3650
@@
 L MIC5219 U?
 U 1 1 58A31A9F
-P 1750 4950
-F 0 "U?" H 1750 5350 60  0000 C CNN
-F 1 "MIC5219" H 1800 4550 60  0000 C CNN
-F 2 "" H 1750 4950 60  0000 C CNN
-F 3 "" H 1750 4950 60  0000 C CNN
-	1    1750 4950
-	1    0    0    -1
-$EndComp
+P 2500 5800
+F 0 "U?" H 2500 6200 60  0000 C CNN
+F 1 "MIC5219" H 2550 5400 60  0000 C CNN
+F 2 "" H 2500 5800 60  0000 C CNN
+F 3 "" H 2500 5800 60  0000 C CNN
+	1    2500 5800
+	1    0    0    -1
+$EndComp
+$Comp
+L CP1 C?
+U 1 1 58A30E2E
+P 1300 5750
+F 0 "C?" H 1325 5850 50  0000 L CNN
+F 1 "CP1" H 1325 5650 50  0000 L CNN
+F 2 "" H 1300 5750 50  0000 C CNN
+F 3 "" H 1300 5750 50  0000 C CNN
+	1    1300 5750
+	1    0    0    -1
+$EndComp
+$Comp
+L CP1 C?
+U 1 1 58A30F4B
+P 3150 5750
+F 0 "C?" H 3175 5850 50  0000 L CNN
+F 1 "CP1" H 3175 5650 50  0000 L CNN
+F 2 "" H 3150 5750 50  0000 C CNN
+F 3 "" H 3150 5750 50  0000 C CNN
+	1    3150 5750
+	1    0    0    -1
+$EndComp
+$Comp
+L C C?
+U 1 1 58A30FC8
+P 3350 5750
+F 0 "C?" H 3375 5850 50  0000 L CNN
+F 1 "C" H 3375 5650 50  0000 L CNN
+F 2 "" H 3388 5600 50  0000 C CNN
+F 3 "" H 3350 5750 50  0000 C CNN
+	1    3350 5750
+	1    0    0    -1
+$EndComp
+$Comp
+L C C?
+U 1 1 58A31059
+P 3550 5750
+F 0 "C?" H 3575 5850 50  0000 L CNN
+F 1 "C" H 3575 5650 50  0000 L CNN
+F 2 "" H 3588 5600 50  0000 C CNN
+F 3 "" H 3550 5750 50  0000 C CNN
+	1    3550 5750
+	1    0    0    -1
+$EndComp
+$Comp
+L LED D?
+U 1 1 58A310F2
+P 3800 6050
+F 0 "D?" H 3800 6150 50  0000 C CNN
+F 1 "LED" H 3800 5950 50  0000 C CNN
+F 2 "" H 3800 6050 50  0000 C CNN
+F 3 "" H 3800 6050 50  0000 C CNN
+	1    3800 6050
+	0    -1   -1   0
+$EndComp
+$Comp
+L R R?
+U 1 1 58A311BF
+P 3800 5750
+F 0 "R?" V 3880 5750 50  0000 C CNN
+F 1 "R" V 3800 5750 50  0000 C CNN
+F 2 "" V 3730 5750 50  0000 C CNN
+F 3 "" H 3800 5750 50  0000 C CNN
+	1    3800 5750
+	1    0    0    -1
+$EndComp
+Wire Wire Line
+	1100 5600 2000 5600
+Wire Wire Line
+	3000 5600 3800 5600
+Connection ~ 3150 5600
+Connection ~ 3350 5600
+$Comp
+L D D?
+U 1 1 58A31E19
+P 1150 5250
+F 0 "D?" H 1150 5350 50  0000 C CNN
+F 1 "D" H 1150 5150 50  0000 C CNN
+F 2 "" H 1150 5250 50  0000 C CNN
+F 3 "" H 1150 5250 50  0000 C CNN
+	1    1150 5250
+	-1   0    0    1
+$EndComp
+Connection ~ 3550 5600
+Wire Wire Line
+	2000 6000 1900 6000
+Wire Wire Line
+	1900 6000 1900 5600
+Connection ~ 1900 5600
+Text GLabel 2400 1600 0    47   Input ~ 0
+RAW
+Text GLabel 1100 5600 0    47   Input ~ 0
+RAW
+Connection ~ 1300 5600
+Text GLabel 1300 5900 3    47   Input ~ 0
+GND
+Text GLabel 1750 5900 3    47   Input ~ 0
+GND
+Text GLabel 3150 5900 3    47   Input ~ 0
+GND
+Text GLabel 3350 5900 3    47   Input ~ 0
+GND
+Text GLabel 3550 5900 3    47   Input ~ 0
+GND
+Wire Wire Line
+	2000 5800 1750 5800
+Wire Wire Line
+	1750 5800 1750 5900
+Text GLabel 3800 6200 3    47   Input ~ 0
+GND
+Wire Wire Line
+	1300 5250 1300 5600
+Text GLabel 3800 5550 1    47   Input ~ 0
+VCC
+Wire Wire Line
+	3800 5600 3800 5550
+$Comp
+L Polyfuse F?
+U 1 1 58A33351
+P 850 5250
+F 0 "F?" V 750 5250 50  0000 C CNN
+F 1 "Polyfuse" V 950 5250 50  0000 C CNN
+F 2 "" H 900 5050 50  0001 L CNN
+F 3 "" H 850 5250 50  0001 C CNN
+	1    850  5250
+	0    1    1    0
+$EndComp
+Text GLabel 600  5000 1    47   Input ~ 0
+UVCC
+Wire Wire Line
+	700  5250 600  5250
+Wire Wire Line
+	600  5250 600  5000
 $EndSCHEMATC
